Commit message: updata g1loco and b2 gait

File: resources/robots/b2z1/b2.urdf (robot description, URDF)
Before this commit: robot b2_description, 37 links, 36 joints
Links:
- link FL_calf: geometry collision box size=0.05 0.028 0.035; collision box size=0.1 0.0245 0.018
- link FL_hip: geometry visual mesh filename=file:///home/zhipy/project/unitree_rl_gym/resources/robots/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
- link FL_thigh: geometry collision box size=0.32 0.0445 0.054; visual mesh filename=file:///home/zhipy/project/unitree_rl_gym/resources/robots/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
- link FR_calf: geometry collision box size=0.05 0.028 0.035; collision box size=0.1 0.0245 0.018
- link FR_hip: mass 2.256 -> 2.673; geometry visual mesh filename=file:///home/zhipy/project/unitree_rl_gym/resources/robots/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
- link FR_thigh: geometry collision box size=0.25 0.028 0.04; visual mesh filename=file:///home/zhipy/project/unitree_rl_gym/resources/robots/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
- link RL_calf: geometry collision box size=0.05 0.028 0.035; collision box size=0.1 0.0245 0.018
- link RL_hip: mass 2.256 -> 2.673; geometry visual mesh filename=file:///home/zhipy/project/unitree_rl_gym/resources/robots/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
- link RL_thigh: geometry collision box size=0.25 0.028 0.04; visual mesh filename=file:///home/zhipy/project/unitree_rl_gym/resources/robots/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
- link RR_calf: geometry collision box size=0.05 0.028 0.035; collision box size=0.1 0.0245 0.018
- link RR_hip: geometry visual mesh filename=file:///home/zhipy/project/unitree_rl_gym/resources/robots/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
- link RR_thigh: geometry collision box size=0.25 0.028 0.04; visual mesh filename=file:///home/zhipy/project/unitree_rl_gym/resources/robots/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
- link base_link: geometry collision box size=0.5 0.28 0.15; visual mesh filename=file:///home/zhipy/project/unitree_rl_gym/resources/robots/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

File: resources/robots/b2z1/b2_description.urdf (robot description, URDF)
Before this commit: robot b2_description, 37 links, 36 joints
Links:
- link FR_hip: mass 2.256 -> 2.673
- link RL_hip: mass 2.256 -> 2.673

File: resources/robots/b2z1/b2z1.urdf (robot description, URDF)
Before this commit: robot b2_description, 47 links, 46 joints
Links:
- link FL_thigh: geometry collision box size=0.25 0.028 0.04; visual mesh filename=./meshes/FL_thigh.dae
- link FR_hip: mass 2.256 -> 2.673
- link RL_hip: mass 2.256 -> 2.673
- link lidar_link: geometry collision box size=0.16 0.152 0.152

File: resources/robots/g1_description/g1_29dof_with_hand_fixed.urdf (robot description, URDF)
Before this commit: robot g1_29dof_with_hand, 53 links, 52 joints
Links:
- link head_link: geometry visual mesh filename=meshes/head_link.STL
- link left_ankle_pitch_link: geometry visual mesh filename=meshes/left_ankle_pitch_link.STL
- link left_ankle_roll_link: geometry collision cylinder length=0.15 radius=0.02; collision cylinder length=0.15 radius=0.02
- link left_elbow_link: geometry collision cylinder length=0.15 radius=0.03; visual mesh filename=meshes/left_elbow_link.STL
- link left_hand_index_0_link: geometry visual mesh filename=meshes/left_hand_index_0_link.STL
- link left_hand_index_1_link: geometry visual mesh filename=meshes/left_hand_index_1_link.STL
- link left_hand_middle_0_link: geometry visual mesh filename=meshes/left_hand_middle_0_link.STL
- link left_hand_middle_1_link: geometry visual mesh filename=meshes/left_hand_middle_1_link.STL
- link left_hand_palm_link: geometry visual mesh filename=meshes/left_hand_palm_link.STL
- link left_hand_thumb_0_link: geometry visual mesh filename=meshes/left_hand_thumb_0_link.STL
- link left_hand_thumb_2_link: geometry visual mesh filename=meshes/left_hand_thumb_2_link.STL
- link left_hip_pitch_link: geometry visual mesh filename=meshes/left_hip_pitch_link.STL
- link left_hip_roll_link: geometry visual mesh filename=meshes/left_hip_roll_link.STL
- link left_hip_yaw_link: geometry collision cylinder length=0.2 radius=0.03; visual mesh filename=meshes/left_hip_yaw_link.STL
- link left_knee_link: geometry collision cylinder length=0.15 radius=0.03; visual mesh filename=meshes/left_knee_link.STL
- link left_shoulder_pitch_link: geometry visual mesh filename=meshes/left_shoulder_pitch_link.STL
- link left_shoulder_yaw_link: geometry collision cylinder length=0.1 radius=0.03; visual mesh filename=meshes/left_shoulder_yaw_link.STL
- link left_wrist_pitch_link: geometry visual mesh filename=meshes/left_wrist_pitch_link.STL
- link left_wrist_roll_link: geometry visual mesh filename=meshes/left_wrist_roll_link.STL
- link left_wrist_yaw_link: geometry visual mesh filename=meshes/left_wrist_yaw_link.STL
- link logo_link: geometry visual mesh filename=meshes/logo_link.STL
- link pelvis_contour_link: geometry visual mesh filename=meshes/pelvis_contour_link.STL
- link right_ankle_pitch_link: geometry visual mesh filename=meshes/right_ankle_pitch_link.STL
- link right_ankle_roll_link: geometry collision cylinder length=0.15 radius=0.02; collision cylinder length=0.15 radius=0.02
- link right_elbow_link: geometry collision cylinder length=0.15 radius=0.03; visual mesh filename=meshes/right_elbow_link.STL
- link right_hand_index_0_link: geometry visual mesh filename=meshes/right_hand_index_0_link.STL
- link right_hand_index_1_link: geometry visual mesh filename=meshes/right_hand_index_1_link.STL
- link right_hand_middle_0_link: geometry visual mesh filename=meshes/right_hand_middle_0_link.STL
- link right_hand_middle_1_link: geometry visual mesh filename=meshes/right_hand_middle_1_link.STL
- link right_hand_palm_link: geometry visual mesh filename=meshes/right_hand_palm_link.STL
- link right_hand_thumb_0_link: geometry visual mesh filename=meshes/right_hand_thumb_0_link.STL
- link right_hand_thumb_2_link: geometry visual mesh filename=meshes/right_hand_thumb_2_link.STL
- link right_hip_pitch_link: geometry visual mesh filename=meshes/right_hip_pitch_link.STL
- link right_hip_roll_link: geometry visual mesh filename=meshes/right_hip_roll_link.STL
- link right_hip_yaw_link: geometry collision cylinder length=0.2 radius=0.03; visual mesh filename=meshes/right_hip_yaw_link.STL
- link right_knee_link: geometry collision cylinder length=0.15 radius=0.03; visual mesh filename=meshes/right_knee_link.STL
- link right_shoulder_pitch_link: geometry visual mesh filename=meshes/right_shoulder_pitch_link.STL
- link right_shoulder_yaw_link: geometry collision cylinder length=0.1 radius=0.03; visual mesh filename=meshes/right_shoulder_yaw_link.STL
- link right_wrist_pitch_link: geometry visual mesh filename=meshes/right_wrist_pitch_link.STL
- link right_wrist_roll_link: geometry visual mesh filename=meshes/right_wrist_roll_link.STL
- link right_wrist_yaw_link: geometry visual mesh filename=meshes/right_wrist_yaw_link.STL
- link torso_link: geometry collision cylinder length=0.35 radius=0.08; visual mesh filename=meshes/torso_link.STL
- link waist_support_link: geometry visual mesh filename=meshes/waist_support_link.STL
