Commit message: 1504

File: resources/robots/b2z1/b2z1.urdf (robot description, URDF)
Before this commit: robot b2_description, 47 links, 46 joints
Links:
- link lidar_link: geometry collision cylinder length=0.16 radius=0.076
Joints:
- joint base_static_joint: origin xyz=-0.05 0. 0.1 rpy=0. 0. 0. -> xyz=0.2 0. 0.225 rpy=0. 0. 0.
