Commit message: update ee and base force control

File: resources/robots/g1_description/g1_29dof_with_hand_fixed_rev_1_0.urdf (robot description, URDF)
Before this commit: robot g1_29dof_with_hand_rev_1_0, 53 links, 52 joints
Links:
- link left_elbow_link: geometry collision box size=0.06 0.06 0.15; visual mesh filename=meshes/left_elbow_link.STL
- link left_hand_thumb_1_link: geometry visual mesh filename=meshes/left_hand_thumb_1_link.STL
- link left_hip_yaw_link: geometry collision box size=0.06 0.06 0.2; visual mesh filename=meshes/left_hip_yaw_link.STL
- link left_knee_link: geometry collision box size=0.06 0.06 0.15; visual mesh filename=meshes/left_knee_link.STL
- link left_shoulder_roll_link: geometry visual mesh filename=meshes/left_shoulder_roll_link.STL
- link left_shoulder_yaw_link: geometry collision box size=0.06 0.06 0.1; visual mesh filename=meshes/left_shoulder_yaw_link.STL
- link right_elbow_link: geometry collision box size=0.06 0.06 0.15; visual mesh filename=meshes/right_elbow_link.STL
- link right_hand_thumb_1_link: geometry visual mesh filename=meshes/right_hand_thumb_1_link.STL
- link right_hip_yaw_link: geometry collision box size=0.06 0.06 0.2; visual mesh filename=meshes/right_hip_yaw_link.STL
- link right_knee_link: geometry collision box size=0.06 0.06 0.15; visual mesh filename=meshes/right_knee_link.STL
- link right_shoulder_roll_link: geometry visual mesh filename=meshes/right_shoulder_roll_link.STL
- link right_shoulder_yaw_link: geometry collision box size=0.06 0.06 0.1; visual mesh filename=meshes/right_shoulder_yaw_link.STL
- link torso_link: geometry collision box size=0.16 0.16 0.35; visual mesh filename=meshes/torso_link_rev_1_0.STL
