Commit message: update pf

File: resources/robots/g1_description/g1_29dof_rev_1_0.urdf (robot description, URDF)
Before this commit: robot g1_29dof_rev_1_0, 39 links, 38 joints
Links:
- link head_link: geometry visual mesh filename=meshes/head_link.STL
- link left_ankle_pitch_link: geometry visual mesh filename=meshes/left_ankle_pitch_link.STL
- link left_ankle_roll_link: geometry collision cylinder length=0.15 radius=0.02; collision cylinder length=0.15 radius=0.02
- link left_elbow_link: geometry collision box size=0.06 0.06 0.06; visual mesh filename=meshes/left_elbow_link.STL
- link left_hip_pitch_link: geometry visual mesh filename=meshes/left_hip_pitch_link.STL
- link left_hip_roll_link: geometry visual mesh filename=meshes/left_hip_roll_link.STL
- link left_hip_yaw_link: geometry collision box size=0.06 0.06 0.2; visual mesh filename=meshes/left_hip_yaw_link.STL
- link left_knee_link: geometry collision box size=0.06 0.06 0.15; visual mesh filename=meshes/left_knee_link.STL
- link left_rubber_hand: geometry visual mesh filename=meshes/left_rubber_hand.STL
- link left_shoulder_pitch_link: geometry visual mesh filename=meshes/left_shoulder_pitch_link.STL
- link left_shoulder_roll_link: geometry visual mesh filename=meshes/left_shoulder_roll_link.STL
- link left_shoulder_yaw_link: geometry collision box size=0.06 0.06 0.2; visual mesh filename=meshes/left_shoulder_yaw_link.STL
- link left_wrist_pitch_link: geometry collision box size=0.06 0.06 0.05; visual mesh filename=meshes/left_wrist_pitch_link.STL
- link left_wrist_roll_link: geometry visual mesh filename=meshes/left_wrist_roll_link.STL
- link left_wrist_yaw_link: geometry visual mesh filename=meshes/left_wrist_yaw_link.STL
- link logo_link: geometry visual mesh filename=meshes/logo_link.STL
- link pelvis: geometry visual mesh filename=meshes/pelvis.STL
- link pelvis_contour_link: geometry visual mesh filename=meshes/pelvis_contour_link.STL
- link right_ankle_pitch_link: geometry visual mesh filename=meshes/right_ankle_pitch_link.STL
- link right_ankle_roll_link: geometry collision cylinder length=0.15 radius=0.02; collision cylinder length=0.15 radius=0.02
- link right_elbow_link: geometry collision box size=0.06 0.06 0.06; visual mesh filename=meshes/right_elbow_link.STL
- link right_hip_pitch_link: geometry visual mesh filename=meshes/right_hip_pitch_link.STL
- link right_hip_roll_link: geometry visual mesh filename=meshes/right_hip_roll_link.STL
- link right_hip_yaw_link: geometry collision box size=0.06 0.06 0.2; visual mesh filename=meshes/right_hip_yaw_link.STL
- link right_knee_link: geometry collision box size=0.06 0.06 0.15; visual mesh filename=meshes/right_knee_link.STL
- link right_rubber_hand: geometry visual mesh filename=meshes/right_rubber_hand.STL
- link right_shoulder_pitch_link: geometry visual mesh filename=meshes/right_shoulder_pitch_link.STL
- link right_shoulder_roll_link: geometry visual mesh filename=meshes/right_shoulder_roll_link.STL
- link right_shoulder_yaw_link: geometry collision box size=0.06 0.06 0.2; visual mesh filename=meshes/right_shoulder_yaw_link.STL
- link right_wrist_pitch_link: geometry collision box size=0.06 0.06 0.05; visual mesh filename=meshes/right_wrist_pitch_link.STL
- link right_wrist_roll_link: geometry visual mesh filename=meshes/right_wrist_roll_link.STL
- link right_wrist_yaw_link: geometry visual mesh filename=meshes/right_wrist_yaw_link.STL
- link torso_link: geometry collision box size=0.16 0.16 0.35; visual mesh filename=meshes/torso_link_rev_1_0.STL
- link waist_roll_link: geometry visual mesh filename=meshes/waist_roll_link_rev_1_0.STL
- link waist_yaw_link: geometry visual mesh filename=meshes/waist_yaw_link_rev_1_0.STL
